File: kicad/Blade.kicad_pcb (KiCad board)
At the start: 2 copper layers, 87.5 x 5 mm, 34 parts, among them J1 Conn_01x01_Male, J2 Conn_01x01_Male, J3 Conn_01x01_Male, J4 Conn_01x01_Male, J5 Conn_01x01_Male, J6 Conn_01x01_Male

Commit message: commit long open changes
Parts:
- added D1: WS2812B-2020, barn53-kicad:WS2812B-2020, F.Cu at (94.5, 136.5)
- added D1: WS2812B-2020, barn53-kicad:WS2812B-2020, F.Cu at (94.5, 126.5)
- added D1: WS2812B-2020, barn53-kicad:WS2812B-2020, F.Cu at (94.5, 116.5)
- added D1: WS2812B-2020, barn53-kicad:WS2812B-2020, F.Cu at (94.5, 111.5)
- added D1: WS2812B-2020, barn53-kicad:WS2812B-2020, F.Cu at (94.5, 106.5)
- added D1: WS2812B-2020, barn53-kicad:WS2812B-2020, F.Cu at (94.5, 121.5)
- added D1: WS2812B-2020, barn53-kicad:WS2812B-2020, F.Cu at (94.5, 131.5)
- added D10: WS2812B-2020, barn53-kicad:WS2812B-2020, F.Cu at (126.0, 126.5)
- added D10: WS2812B-2020, barn53-kicad:WS2812B-2020, F.Cu at (126.0, 116.5)
- added D10: WS2812B-2020, barn53-kicad:WS2812B-2020, F.Cu at (126.0, 111.5)
- added D10: WS2812B-2020, barn53-kicad:WS2812B-2020, F.Cu at (126.0, 106.5)
- added D10: WS2812B-2020, barn53-kicad:WS2812B-2020, F.Cu at (126.0, 121.5)
- added D10: WS2812B-2020, barn53-kicad:WS2812B-2020, F.Cu at (126.0, 136.5)
- added D10: WS2812B-2020, barn53-kicad:WS2812B-2020, F.Cu at (126.0, 131.5)
- added D11: WS2812B-2020, barn53-kicad:WS2812B-2020, F.Cu at (129.5, 111.5)
- added D11: WS2812B-2020, barn53-kicad:WS2812B-2020, F.Cu at (129.5, 121.5)
- added D11: WS2812B-2020, barn53-kicad:WS2812B-2020, F.Cu at (129.5, 106.5)
- added D11: WS2812B-2020, barn53-kicad:WS2812B-2020, F.Cu at (129.5, 116.5)
- added D11: WS2812B-2020, barn53-kicad:WS2812B-2020, F.Cu at (129.5, 136.5)
- added D11: WS2812B-2020, barn53-kicad:WS2812B-2020, F.Cu at (129.5, 131.5)
- added D11: WS2812B-2020, barn53-kicad:WS2812B-2020, F.Cu at (129.5, 126.5)
- added D12: WS2812B-2020, barn53-kicad:WS2812B-2020, F.Cu at (133.0, 136.5)
- added D12: WS2812B-2020, barn53-kicad:WS2812B-2020, F.Cu at (133.0, 116.5)
- added D12: WS2812B-2020, barn53-kicad:WS2812B-2020, F.Cu at (133.0, 111.5)
- added D12: WS2812B-2020, barn53-kicad:WS2812B-2020, F.Cu at (133.0, 131.5)
- added D12: WS2812B-2020, barn53-kicad:WS2812B-2020, F.Cu at (133.0, 126.5)
- added D12: WS2812B-2020, barn53-kicad:WS2812B-2020, F.Cu at (133.0, 106.5)
- added D12: WS2812B-2020, barn53-kicad:WS2812B-2020, F.Cu at (133.0, 121.5)
- added D13: WS2812B-2020, barn53-kicad:WS2812B-2020, F.Cu at (136.5, 111.5)
- added D13: WS2812B-2020, barn53-kicad:WS2812B-2020, F.Cu at (136.5, 106.5)
- added D13: WS2812B-2020, barn53-kicad:WS2812B-2020, F.Cu at (136.5, 136.5)
- added D13: WS2812B-2020, barn53-kicad:WS2812B-2020, F.Cu at (136.5, 116.5)
- added D13: WS2812B-2020, barn53-kicad:WS2812B-2020, F.Cu at (136.5, 126.5)
- added D13: WS2812B-2020, barn53-kicad:WS2812B-2020, F.Cu at (136.5, 121.5)
- added D13: WS2812B-2020, barn53-kicad:WS2812B-2020, F.Cu at (136.5, 131.5)
- added D14: WS2812B-2020, barn53-kicad:WS2812B-2020, F.Cu at (140.0, 136.5)
- added D14: WS2812B-2020, barn53-kicad:WS2812B-2020, F.Cu at (140.0, 131.5)
- added D14: WS2812B-2020, barn53-kicad:WS2812B-2020, F.Cu at (140.0, 111.5)
- added D14: WS2812B-2020, barn53-kicad:WS2812B-2020, F.Cu at (140.0, 116.5)
- added D14: WS2812B-2020, barn53-kicad:WS2812B-2020, F.Cu at (140.0, 126.5)
- added D14: WS2812B-2020, barn53-kicad:WS2812B-2020, F.Cu at (140.0, 121.5)
- added D14: WS2812B-2020, barn53-kicad:WS2812B-2020, F.Cu at (140.0, 106.5)
- added D15: WS2812B-2020, barn53-kicad:WS2812B-2020, F.Cu at (143.5, 136.5)
- added D15: WS2812B-2020, barn53-kicad:WS2812B-2020, F.Cu at (143.5, 126.5)
- added D15: WS2812B-2020, barn53-kicad:WS2812B-2020, F.Cu at (143.5, 121.5)
- added D15: WS2812B-2020, barn53-kicad:WS2812B-2020, F.Cu at (143.5, 116.5)
- added D15: WS2812B-2020, barn53-kicad:WS2812B-2020, F.Cu at (143.5, 111.5)
- added D15: WS2812B-2020, barn53-kicad:WS2812B-2020, F.Cu at (143.5, 131.5)
- added D15: WS2812B-2020, barn53-kicad:WS2812B-2020, F.Cu at (143.5, 106.5)
- added D16: WS2812B-2020, barn53-kicad:WS2812B-2020, F.Cu at (147.0, 131.5)
- added D16: WS2812B-2020, barn53-kicad:WS2812B-2020, F.Cu at (147.0, 111.5)
- added D16: WS2812B-2020, barn53-kicad:WS2812B-2020, F.Cu at (147.0, 121.5)
- added D16: WS2812B-2020, barn53-kicad:WS2812B-2020, F.Cu at (147.0, 116.5)
- added D16: WS2812B-2020, barn53-kicad:WS2812B-2020, F.Cu at (147.0, 126.5)
- added D16: WS2812B-2020, barn53-kicad:WS2812B-2020, F.Cu at (147.0, 106.5)
- added D16: WS2812B-2020, barn53-kicad:WS2812B-2020, F.Cu at (147.0, 136.5)
- added D17: WS2812B-2020, barn53-kicad:WS2812B-2020, F.Cu at (150.5, 126.5)
- added D17: WS2812B-2020, barn53-kicad:WS2812B-2020, F.Cu at (150.5, 136.5)
- added D17: WS2812B-2020, barn53-kicad:WS2812B-2020, F.Cu at (150.5, 116.5)
- added D17: WS2812B-2020, barn53-kicad:WS2812B-2020, F.Cu at (150.5, 121.5)
- added D17: WS2812B-2020, barn53-kicad:WS2812B-2020, F.Cu at (150.5, 131.5)
- added D17: WS2812B-2020, barn53-kicad:WS2812B-2020, F.Cu at (150.5, 111.5)
- added D17: WS2812B-2020, barn53-kicad:WS2812B-2020, F.Cu at (150.5, 106.5)
- added D18: WS2812B-2020, barn53-kicad:WS2812B-2020, F.Cu at (154.0, 131.5)
- added D18: WS2812B-2020, barn53-kicad:WS2812B-2020, F.Cu at (154.0, 111.5)
- added D18: WS2812B-2020, barn53-kicad:WS2812B-2020, F.Cu at (154.0, 126.5)
- added D18: WS2812B-2020, barn53-kicad:WS2812B-2020, F.Cu at (154.0, 106.5)
- added D18: WS2812B-2020, barn53-kicad:WS2812B-2020, F.Cu at (154.0, 136.5)
- added D18: WS2812B-2020, barn53-kicad:WS2812B-2020, F.Cu at (154.0, 121.5)
- added D18: WS2812B-2020, barn53-kicad:WS2812B-2020, F.Cu at (154.0, 116.5)
- added D19: WS2812B-2020, barn53-kicad:WS2812B-2020, F.Cu at (157.5, 106.5)
- added D19: WS2812B-2020, barn53-kicad:WS2812B-2020, F.Cu at (157.5, 131.5)
- added D19: WS2812B-2020, barn53-kicad:WS2812B-2020, F.Cu at (157.5, 121.5)
- added D19: WS2812B-2020, barn53-kicad:WS2812B-2020, F.Cu at (157.5, 116.5)
- added D19: WS2812B-2020, barn53-kicad:WS2812B-2020, F.Cu at (157.5, 126.5)
- added D19: WS2812B-2020, barn53-kicad:WS2812B-2020, F.Cu at (157.5, 111.5)
- added D19: WS2812B-2020, barn53-kicad:WS2812B-2020, F.Cu at (157.5, 136.5)
- added D2: WS2812B-2020, barn53-kicad:WS2812B-2020, F.Cu at (98.0, 136.5)
- added D2: WS2812B-2020, barn53-kicad:WS2812B-2020, F.Cu at (98.0, 121.5)
- added D2: WS2812B-2020, barn53-kicad:WS2812B-2020, F.Cu at (98.0, 111.5)
- added D2: WS2812B-2020, barn53-kicad:WS2812B-2020, F.Cu at (98.0, 106.5)
- added D2: WS2812B-2020, barn53-kicad:WS2812B-2020, F.Cu at (98.0, 131.5)
- added D2: WS2812B-2020, barn53-kicad:WS2812B-2020, F.Cu at (98.0, 126.5)
- added D2: WS2812B-2020, barn53-kicad:WS2812B-2020, F.Cu at (98.0, 116.5)
- added D20: WS2812B-2020, barn53-kicad:WS2812B-2020, F.Cu at (161.0, 136.5)
- added D20: WS2812B-2020, barn53-kicad:WS2812B-2020, F.Cu at (161.0, 121.5)
- added D20: WS2812B-2020, barn53-kicad:WS2812B-2020, F.Cu at (161.0, 116.5)
- added D20: WS2812B-2020, barn53-kicad:WS2812B-2020, F.Cu at (161.0, 111.5)
- added D20: WS2812B-2020, barn53-kicad:WS2812B-2020, F.Cu at (161.0, 106.5)
- added D20: WS2812B-2020, barn53-kicad:WS2812B-2020, F.Cu at (161.0, 131.5)
- added D20: WS2812B-2020, barn53-kicad:WS2812B-2020, F.Cu at (161.0, 126.5)
- added D21: WS2812B-2020, barn53-kicad:WS2812B-2020, F.Cu at (164.5, 136.5)
- added D21: WS2812B-2020, barn53-kicad:WS2812B-2020, F.Cu at (164.5, 131.5)
- added D21: WS2812B-2020, barn53-kicad:WS2812B-2020, F.Cu at (164.5, 111.5)
- added D21: WS2812B-2020, barn53-kicad:WS2812B-2020, F.Cu at (164.5, 121.5)
- added D21: WS2812B-2020, barn53-kicad:WS2812B-2020, F.Cu at (164.5, 126.5)
- added D21: WS2812B-2020, barn53-kicad:WS2812B-2020, F.Cu at (164.5, 106.5)
- added D21: WS2812B-2020, barn53-kicad:WS2812B-2020, F.Cu at (164.5, 116.5)
- added D22: WS2812B-2020, barn53-kicad:WS2812B-2020, F.Cu at (168.0, 116.5)
- added D22: WS2812B-2020, barn53-kicad:WS2812B-2020, F.Cu at (168.0, 131.5)
- added D22: WS2812B-2020, barn53-kicad:WS2812B-2020, F.Cu at (168.0, 106.5)
- added D22: WS2812B-2020, barn53-kicad:WS2812B-2020, F.Cu at (168.0, 121.5)
- added D22: WS2812B-2020, barn53-kicad:WS2812B-2020, F.Cu at (168.0, 136.5)
- added D22: WS2812B-2020, barn53-kicad:WS2812B-2020, F.Cu at (168.0, 126.5)
- added D22: WS2812B-2020, barn53-kicad:WS2812B-2020, F.Cu at (168.0, 111.5)
- added D23: WS2812B-2020, barn53-kicad:WS2812B-2020, F.Cu at (171.5, 136.5)
- added D23: WS2812B-2020, barn53-kicad:WS2812B-2020, F.Cu at (171.5, 121.5)
- added D23: WS2812B-2020, barn53-kicad:WS2812B-2020, F.Cu at (171.5, 126.5)
- added D23: WS2812B-2020, barn53-kicad:WS2812B-2020, F.Cu at (171.5, 131.5)
- added D23: WS2812B-2020, barn53-kicad:WS2812B-2020, F.Cu at (171.5, 111.5)
- added D23: WS2812B-2020, barn53-kicad:WS2812B-2020, F.Cu at (171.5, 116.5)
- added D23: WS2812B-2020, barn53-kicad:WS2812B-2020, F.Cu at (171.5, 106.5)
- added D24: WS2812B-2020, barn53-kicad:WS2812B-2020, F.Cu at (175.0, 121.5)
- added D24: WS2812B-2020, barn53-kicad:WS2812B-2020, F.Cu at (175.0, 111.5)
- added D24: WS2812B-2020, barn53-kicad:WS2812B-2020, F.Cu at (175.0, 131.5)
- added D24: WS2812B-2020, barn53-kicad:WS2812B-2020, F.Cu at (175.0, 106.5)
- added D24: WS2812B-2020, barn53-kicad:WS2812B-2020, F.Cu at (175.0, 136.5)
- added D24: WS2812B-2020, barn53-kicad:WS2812B-2020, F.Cu at (175.0, 116.5)
- added D24: WS2812B-2020, barn53-kicad:WS2812B-2020, F.Cu at (175.0, 126.5)
- added D25: WS2812B-2020, barn53-kicad:WS2812B-2020, F.Cu at (178.5, 106.5)
- added D25: WS2812B-2020, barn53-kicad:WS2812B-2020, F.Cu at (178.5, 136.5)
- added D25: WS2812B-2020, barn53-kicad:WS2812B-2020, F.Cu at (178.5, 111.5)
- added D25: WS2812B-2020, barn53-kicad:WS2812B-2020, F.Cu at (178.5, 131.5)
- added D25: WS2812B-2020, barn53-kicad:WS2812B-2020, F.Cu at (178.5, 126.5)
- added D25: WS2812B-2020, barn53-kicad:WS2812B-2020, F.Cu at (178.5, 121.5)
- added D25: WS2812B-2020, barn53-kicad:WS2812B-2020, F.Cu at (178.5, 116.5)
- added D3: WS2812B-2020, barn53-kicad:WS2812B-2020, F.Cu at (101.5, 106.5)
- added D3: WS2812B-2020, barn53-kicad:WS2812B-2020, F.Cu at (101.5, 126.5)
- added D3: WS2812B-2020, barn53-kicad:WS2812B-2020, F.Cu at (101.5, 136.5)
- added D3: WS2812B-2020, barn53-kicad:WS2812B-2020, F.Cu at (101.5, 116.5)
- added D3: WS2812B-2020, barn53-kicad:WS2812B-2020, F.Cu at (101.5, 111.5)
- added D3: WS2812B-2020, barn53-kicad:WS2812B-2020, F.Cu at (101.5, 121.5)
- added D3: WS2812B-2020, barn53-kicad:WS2812B-2020, F.Cu at (101.5, 131.5)
- added D4: WS2812B-2020, barn53-kicad:WS2812B-2020, F.Cu at (105.0, 106.5)
- added D4: WS2812B-2020, barn53-kicad:WS2812B-2020, F.Cu at (105.0, 136.5)
- added D4: WS2812B-2020, barn53-kicad:WS2812B-2020, F.Cu at (105.0, 116.5)
- added D4: WS2812B-2020, barn53-kicad:WS2812B-2020, F.Cu at (105.0, 126.5)
- added D4: WS2812B-2020, barn53-kicad:WS2812B-2020, F.Cu at (105.0, 131.5)
- added D4: WS2812B-2020, barn53-kicad:WS2812B-2020, F.Cu at (105.0, 121.5)
- added D4: WS2812B-2020, barn53-kicad:WS2812B-2020, F.Cu at (105.0, 111.5)
- added D5: WS2812B-2020, barn53-kicad:WS2812B-2020, F.Cu at (108.5, 126.5)
- added D5: WS2812B-2020, barn53-kicad:WS2812B-2020, F.Cu at (108.5, 106.5)
- added D5: WS2812B-2020, barn53-kicad:WS2812B-2020, F.Cu at (108.5, 111.5)
- added D5: WS2812B-2020, barn53-kicad:WS2812B-2020, F.Cu at (108.5, 116.5)
- added D5: WS2812B-2020, barn53-kicad:WS2812B-2020, F.Cu at (108.5, 131.5)
- added D5: WS2812B-2020, barn53-kicad:WS2812B-2020, F.Cu at (108.5, 121.5)
- added D5: WS2812B-2020, barn53-kicad:WS2812B-2020, F.Cu at (108.5, 136.5)
- added D6: WS2812B-2020, barn53-kicad:WS2812B-2020, F.Cu at (112.0, 121.5)
- added D6: WS2812B-2020, barn53-kicad:WS2812B-2020, F.Cu at (112.0, 126.5)
- added D6: WS2812B-2020, barn53-kicad:WS2812B-2020, F.Cu at (112.0, 111.5)
- added D6: WS2812B-2020, barn53-kicad:WS2812B-2020, F.Cu at (112.0, 116.5)
- added D6: WS2812B-2020, barn53-kicad:WS2812B-2020, F.Cu at (112.0, 106.5)
- added D6: WS2812B-2020, barn53-kicad:WS2812B-2020, F.Cu at (112.0, 131.5)
- added D6: WS2812B-2020, barn53-kicad:WS2812B-2020, F.Cu at (112.0, 136.5)
- added D7: WS2812B-2020, barn53-kicad:WS2812B-2020, F.Cu at (115.5, 111.5)
- added D7: WS2812B-2020, barn53-kicad:WS2812B-2020, F.Cu at (115.5, 131.5)
- added D7: WS2812B-2020, barn53-kicad:WS2812B-2020, F.Cu at (115.5, 136.5)
- added D7: WS2812B-2020, barn53-kicad:WS2812B-2020, F.Cu at (115.5, 121.5)
- added D7: WS2812B-2020, barn53-kicad:WS2812B-2020, F.Cu at (115.5, 106.5)
- added D7: WS2812B-2020, barn53-kicad:WS2812B-2020, F.Cu at (115.5, 126.5)
- added D7: WS2812B-2020, barn53-kicad:WS2812B-2020, F.Cu at (115.5, 116.5)
- added D8: WS2812B-2020, barn53-kicad:WS2812B-2020, F.Cu at (119.0, 136.5)
- added D8: WS2812B-2020, barn53-kicad:WS2812B-2020, F.Cu at (119.0, 131.5)
- added D8: WS2812B-2020, barn53-kicad:WS2812B-2020, F.Cu at (119.0, 126.5)
- added D8: WS2812B-2020, barn53-kicad:WS2812B-2020, F.Cu at (119.0, 111.5)
- added D8: WS2812B-2020, barn53-kicad:WS2812B-2020, F.Cu at (119.0, 106.5)
- added D8: WS2812B-2020, barn53-kicad:WS2812B-2020, F.Cu at (119.0, 116.5)
- added D8: WS2812B-2020, barn53-kicad:WS2812B-2020, F.Cu at (119.0, 121.5)
- added D9: WS2812B-2020, barn53-kicad:WS2812B-2020, F.Cu at (122.5, 131.5)
- added D9: WS2812B-2020, barn53-kicad:WS2812B-2020, F.Cu at (122.5, 121.5)
- added D9: WS2812B-2020, barn53-kicad:WS2812B-2020, F.Cu at (122.5, 116.5)
- added D9: WS2812B-2020, barn53-kicad:WS2812B-2020, F.Cu at (122.5, 126.5)
- added D9: WS2812B-2020, barn53-kicad:WS2812B-2020, F.Cu at (122.5, 106.5)
- added D9: WS2812B-2020, barn53-kicad:WS2812B-2020, F.Cu at (122.5, 111.5)
- added D9: WS2812B-2020, barn53-kicad:WS2812B-2020, F.Cu at (122.5, 136.5)
- added J1: Conn_01x01_Male, barn53-kicad:PCBSolderConnector_1x0.7, B.Cu at (93.3, 127.5)
- added J1: Conn_01x01_Male, barn53-kicad:PCBSolderConnector_1x0.7, B.Cu at (93.3, 112.5)
- added J1: Conn_01x01_Male, barn53-kicad:PCBSolderConnector_1x0.7, B.Cu at (93.3, 137.5)
- added J1: Conn_01x01_Male, barn53-kicad:PCBSolderConnector_1x0.7, B.Cu at (93.3, 132.5)
- added J1: Conn_01x01_Male, barn53-kicad:PCBSolderConnector_1x0.7, B.Cu at (93.3, 122.5)
- added J1: Conn_01x01_Male, barn53-kicad:PCBSolderConnector_1x0.7, B.Cu at (93.3, 117.5)
- added J1: Conn_01x01_Male, barn53-kicad:PCBSolderConnector_1x0.7, B.Cu at (93.3, 107.5)
- added J2: Conn_01x01_Male, barn53-kicad:PCBSolderConnector_1x0.7, B.Cu at (179.8, 137.5)
- added J2: Conn_01x01_Male, barn53-kicad:PCBSolderConnector_1x0.7, B.Cu at (179.8, 132.5)
- added J2: Conn_01x01_Male, barn53-kicad:PCBSolderConnector_1x0.7, B.Cu at (179.8, 127.5)
- added J2: Conn_01x01_Male, barn53-kicad:PCBSolderConnector_1x0.7, B.Cu at (179.8, 122.5)
- added J2: Conn_01x01_Male, barn53-kicad:PCBSolderConnector_1x0.7, B.Cu at (179.8, 112.5)
- added J2: Conn_01x01_Male, barn53-kicad:PCBSolderConnector_1x0.7, B.Cu at (179.8, 107.5)
- added J2: Conn_01x01_Male, barn53-kicad:PCBSolderConnector_1x0.7, B.Cu at (179.8, 117.5)
- added J3: Conn_01x01_Male, barn53-kicad:PCBSolderConnector_1x0.7, B.Cu at (93.3, 106.5)
- added J3: Conn_01x01_Male, barn53-kicad:PCBSolderConnector_1x0.7, B.Cu at (93.3, 121.5)
- added J3: Conn_01x01_Male, barn53-kicad:PCBSolderConnector_1x0.7, B.Cu at (93.3, 111.5)
- added J3: Conn_01x01_Male, barn53-kicad:PCBSolderConnector_1x0.7, B.Cu at (93.3, 126.5)
- added J3: Conn_01x01_Male, barn53-kicad:PCBSolderConnector_1x0.7, B.Cu at (93.3, 116.5)
- added J3: Conn_01x01_Male, barn53-kicad:PCBSolderConnector_1x0.7, B.Cu at (93.3, 136.5)
- added J3: Conn_01x01_Male, barn53-kicad:PCBSolderConnector_1x0.7, B.Cu at (93.3, 131.5)
- added J4: Conn_01x01_Male, barn53-kicad:PCBSolderConnector_1x0.7, B.Cu at (179.8, 106.5)
- added J4: Conn_01x01_Male, barn53-kicad:PCBSolderConnector_1x0.7, B.Cu at (179.8, 111.5)
- added J4: Conn_01x01_Male, barn53-kicad:PCBSolderConnector_1x0.7, B.Cu at (179.8, 116.5)
- added J4: Conn_01x01_Male, barn53-kicad:PCBSolderConnector_1x0.7, B.Cu at (179.8, 136.5)
- added J4: Conn_01x01_Male, barn53-kicad:PCBSolderConnector_1x0.7, B.Cu at (179.8, 131.5)
- added J4: Conn_01x01_Male, barn53-kicad:PCBSolderConnector_1x0.7, B.Cu at (179.8, 126.5)
- added J4: Conn_01x01_Male, barn53-kicad:PCBSolderConnector_1x0.7, B.Cu at (179.8, 121.5)
- added J5: Conn_01x01_Male, barn53-kicad:PCBSolderConnector_1x0.7, B.Cu at (179.8, 120.5)
- added J5: Conn_01x01_Male, barn53-kicad:PCBSolderConnector_1x0.7, B.Cu at (179.8, 105.5)
- added J5: Conn_01x01_Male, barn53-kicad:PCBSolderConnector_1x0.7, B.Cu at (179.8, 125.5)
- added J5: Conn_01x01_Male, barn53-kicad:PCBSolderConnector_1x0.7, B.Cu at (179.8, 135.5)
- added J5: Conn_01x01_Male, barn53-kicad:PCBSolderConnector_1x0.7, B.Cu at (179.8, 115.5)
- added J5: Conn_01x01_Male, barn53-kicad:PCBSolderConnector_1x0.7, B.Cu at (179.8, 130.5)
- added J5: Conn_01x01_Male, barn53-kicad:PCBSolderConnector_1x0.7, B.Cu at (179.8, 110.5)
- added J6: Conn_01x01_Male, barn53-kicad:PCBSolderConnector_1x0.7, B.Cu at (93.3, 105.5)
- added J6: Conn_01x01_Male, barn53-kicad:PCBSolderConnector_1x0.7, B.Cu at (93.3, 130.5)
- added J6: Conn_01x01_Male, barn53-kicad:PCBSolderConnector_1x0.7, B.Cu at (93.3, 135.5)
- added J6: Conn_01x01_Male, barn53-kicad:PCBSolderConnector_1x0.7, B.Cu at (93.3, 115.5)
- added J6: Conn_01x01_Male, barn53-kicad:PCBSolderConnector_1x0.7, B.Cu at (93.3, 110.5)
- added J6: Conn_01x01_Male, barn53-kicad:PCBSolderConnector_1x0.7, B.Cu at (93.3, 125.5)
- added J6: Conn_01x01_Male, barn53-kicad:PCBSolderConnector_1x0.7, B.Cu at (93.3, 120.5)
- added REF**: Breakaway Tab, barn53-kicad:Breakaway Tab, F.Cu at (134.6, 133.0)
- added REF**: Breakaway Tab, barn53-kicad:Breakaway Tab, F.Cu at (134.6, 113.0)
- added REF**: Breakaway Tab, barn53-kicad:Breakaway Tab, F.Cu at (134.6, 108.0)
- added REF**: Breakaway Tab, barn53-kicad:Breakaway Tab, F.Cu at (170.8, 108.0)
- added REF**: Breakaway Tab, barn53-kicad:Breakaway Tab, F.Cu at (134.6, 118.0)
- added REF**: Breakaway Tab, barn53-kicad:Breakaway Tab, F.Cu at (170.8, 133.0)
- added REF**: Breakaway Tab, barn53-kicad:Breakaway Tab, F.Cu at (170.8, 123.0)
- added REF**: Breakaway Tab, barn53-kicad:Breakaway Tab, F.Cu at (134.6, 123.0)
- added REF**: Breakaway Tab, barn53-kicad:Breakaway Tab, F.Cu at (170.8, 118.0)
- added REF**: Breakaway Tab, barn53-kicad:Breakaway Tab, F.Cu at (134.6, 128.0)
- added REF**: Breakaway Tab, barn53-kicad:Breakaway Tab, F.Cu at (170.8, 113.0)
- added REF**: Breakaway Tab, barn53-kicad:Breakaway Tab, F.Cu at (98.3, 108.0)
- added REF**: Breakaway Tab, barn53-kicad:Breakaway Tab, F.Cu at (98.3, 118.0)
- added REF**: Breakaway Tab, barn53-kicad:Breakaway Tab, F.Cu at (98.3, 113.0)
- added REF**: Breakaway Tab, barn53-kicad:Breakaway Tab, F.Cu at (98.3, 133.0)
- added REF**: Breakaway Tab, barn53-kicad:Breakaway Tab, F.Cu at (98.3, 123.0)
- added REF**: Breakaway Tab, barn53-kicad:Breakaway Tab, F.Cu at (98.3, 128.0)
- added REF**: Breakaway Tab, barn53-kicad:Breakaway Tab, F.Cu at (170.8, 128.0)
Routing:
- net +3V3: track 90.6 -> 880.4 mm, vias 4 -> 200
- net GND: track 86.8 -> 694.1 mm, vias 3 -> 200
- net /Dout: track 2.31 -> 18.5 mm, vias 1 -> 8
- net /Din: track 2.31 -> 18.5 mm, vias 1 -> 8
- net Net-(D8-Pad1): track 2.01 -> 16.1 mm
- net Net-(D7-Pad1): track 2.01 -> 16.1 mm
- net Net-(D6-Pad1): track 2.01 -> 16.1 mm
- net Net-(D4-Pad1): track 2.01 -> 16.1 mm
- net Net-(D3-Pad1): track 2.01 -> 16.1 mm
- net Net-(D24-Pad1): track 2.01 -> 16.1 mm
- net Net-(D23-Pad1): track 2.01 -> 16.1 mm
- net Net-(D22-Pad1): track 2.01 -> 16.1 mm
- net Net-(D21-Pad1): track 2.01 -> 16.1 mm
- net Net-(D20-Pad1): track 2.01 -> 16.1 mm
- net Net-(D2-Pad1): track 2.01 -> 16.1 mm
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Other:
- board size 87.5 x 5 mm -> 87.5 x 38 mm
